File: BenchBudEE.sch (KiCad schematic (older format))
At the start: 0 parts

Commit message: Arduino module
Changed lines of the file:
@@
-EESchema Schematic File Version 2  date 2/8/2014 12:16:58 PM
+EESchema Schematic File Version 2  date 2/9/2014 9:38:42 PM
 LIBS:power
 LIBS:device
@@
 Sheet 1 9
 Title ""
-Date "8 feb 2014"
+Date "10 feb 2014"
 Rev ""
 Comp ""
@@
 $EndDescr
 $Sheet
-S 1550 4500 1300 2150
+S 1650 3450 1350 2800
 U 52F19D5D
 F0 "Arduino" 50
 F1 "Arduino.sch" 50
-F2 "Relay-" I R 2850 6400 60
-F3 "MOSI" O R 2850 5450 60
-F4 "MISO" I R 2850 5650 60
-F5 "SCLK" O R 2850 5800 60
-F6 "CS_N" O R 2850 5950 60
-F7 "LED_EN" O R 2850 4900 60
-F8 "LED_Freq" O R 2850 5050 60
-F9 "FAN_EN" O R 2850 4600 60
-F10 "TACH_MEAS" I R 2850 4750 60
-F11 "Relay+" O R 2850 6200 60
-$EndSheet
-$Sheet
-S 7700 3850 1650 1150
+F2 "Relay-" I R 3000 6000 60
+F3 "MOSI" O R 3000 4600 60
+F4 "MISO" I R 3000 4750 60
+F5 "SCLK" O R 3000 5050 60
+F6 "TACH_MEAS" I R 3000 5400 60
+F7 "Relay+" O R 3000 5850 60
+F8 "CURR_MEAS" I R 3000 5300 60
+F9 "FAN_EN_N" O R 3000 4400 60
+F10 "DAC_CS_N" O R 3000 4900 60
+F11 "V+_ADJ_MON" I R 3000 3950 60
+F12 "V-_ADJ_MON" I R 3000 4100 60
+F13 "LED_EN_PWM" O R 3000 5700 60
+F14 "ADC_CS_N" O R 3000 5550 60
+$EndSheet
+$Sheet
+S 7700 3800 1650 1150
 U 52F19DA7
 F0 "Thermocouple" 50
 F1 "Thermocouple.sch" 50
-F2 "TC IN +" I R 9350 4150 60
-F3 "TC IN -" I R 9350 4400 60
-F4 "MOSI" I L 7700 4100 60
-F5 "MISO" O L 7700 4250 60
-F6 "SCLK" I L 7700 4450 60
-F7 "CS_N" I L 7700 4600 60
-$EndSheet
-$Sheet
-S 7700 5400 1700 1300
+F2 "TC IN +" I R 9350 4100 60
+F3 "TC IN -" I R 9350 4350 60
+F4 "MOSI" I L 7700 4050 60
+F5 "MISO" O L 7700 4200 60
+F6 "SCLK" I L 7700 4400 60
+F7 "CS_N" I L 7700 4550 60
+$EndSheet
+$Sheet
+S 7700 6200 1750 700
 U 52F19DBB
 F0 "Relay" 50
 F1 "Relay.sch" 50
-F2 "Din +" I L 7700 5700 60
-F3 "Din -" O L 7700 6000 60
-F4 "NC" B R 9400 5800 60
-F5 "NO" B R 9400 6050 60
-F6 "COM" B R 9400 5550 60
+F2 "RELAY_NC" B R 9450 6550 60
+F3 "RELAY_NO" B R 9450 6700 60
+F4 "RELAY_COM" B R 9450 6400 60
+F5 "RELAY_+" I L 7700 6400 60
+F6 "RELAY_-" O L 7700 6600 60
 $EndSheet
 $Sheet
@@
 $EndSheet
 $Sheet
-S 7700 750  1450 1150
+S 10000 1300 1050 5600
+U 52F19E3F
+F0 "TerminalBlock" 50
+F1 "TerminalBlock.sch" 50
+F2 "V+_ADJ" O L 10000 1700 60
+F3 "V-_ADJ" O L 10000 1850 60
+F4 "FAN_OUT+" O L 10000 2650 60
+F5 "FAN_OUT-" O L 10000 2800 60
+F6 "LED_STRING+" O L 10000 5300 60
+F7 "LED_STRING-" O L 10000 5450 60
+F8 "RELAY_COM" B L 10000 6400 60
+F9 "REALAY_NO" B L 10000 6700 60
+F10 "RELAY_NC" B L 10000 6550 60
+F11 "TACH_IN" I L 10000 3350 60
+F12 "TC_IN+" I L 10000 4100 60
+F13 "TC_IN-" I L 10000 4350 60
+$EndSheet
+$Sheet
+S 7700 5150 1700 750
+U 52F19DF1
+F0 "Led_Driver" 50
+F1 "Led_Driver.sch" 50
+F2 "LED_EN_PWM" I L 7700 5400 60
+F3 "LED_String+" O R 9400 5300 60
+F4 "LED_String-" O R 9400 5450 60
+$EndSheet
+$Sheet
+S 4250 1000 1500 1150
+U 52F64696
+F0 "PowerAdjustmentMonitor" 50
+F1 "PowerAdjustmentMonitor.sch" 50
+F2 "V+_ADJ" O R 5750 1700 60
+F3 "V-_ADJ" O R 5750 1850 60
+F4 "3V3_MON" O L 4250 1250 60
+F5 "5V_MON" O L 4250 1100 60
+F6 "V+_ADJ_MON" O L 4250 1900 60
+F7 "V-_ADJ_MON" O L 4250 2050 60
+F8 "V-_CURR_MON" O L 4250 1650 60
+F9 "V+_CURR_MON" O L 4250 1500 60
+$EndSheet
+$Sheet
+S 7650 2450 1450 1150
 U 52F19E13
 F0 "Fan" 50
 F1 "Fan.sch" 50
-F2 "Power+" O R 9150 1000 60
-F3 "Power-" I R 9150 1150 60
-F4 "Tach" I R 9150 1300 60
-F5 "TachOUT" O L 7700 1750 60
-F6 "FanIn" I L 7700 900 60
-F7 "Current Measure" O L 7700 1650 60
-F8 "MISO" O L 7700 1150 60
-F9 "MOSI" I L 7700 1050 60
-F10 "SCLK" I L 7700 1250 60
-$EndSheet
-$Sheet
-S 10000 1300 1000 5200
-U 52F19E3F
-F0 "TerminalBlock" 50
-F1 "TerminalBlock.sch" 50
-$EndSheet
-$Sheet
-S 7700 2150 1700 1300
-U 52F19DF1
-F0 "Led_Driver" 50
-F1 "Led_Driver.sch" 50
-F2 "EN" I L 7700 2400 60
-F3 "FREQ" I L 7700 2750 60
-F4 "Strig+" O R 9400 2500 60
-F5 "String-" I R 9400 2750 60
-$EndSheet
-$Sheet
-S 4100 1100 1500 1150
-U 52F64696
-F0 "PowerAdjustmentMonitor" 50
-F1 "PowerAdjustmentMonitor.sch" 50
-$EndSheet
+F2 "Current Measure" O L 7650 3450 60
+F3 "MISO" O L 7650 2850 60
+F4 "MOSI" I L 7650 2750 60
+F5 "SCLK" I L 7650 3050 60
+F6 "FAN_OUT_+" O R 9100 2650 60
+F7 "TACH_MEAS_" O L 7650 3350 60
+F8 "FAN_EN_N" I L 7650 2550 60
+F9 "CS_N" I L 7650 2950 60
+F10 "FAN_OUT-" O R 9100 2800 60
+F11 "TACH_IN" I R 9100 3350 60
+$EndSheet
+Wire Wire Line
+	10000 1700 5750 1700
+Wire Wire Line
+	5750 1850 10000 1850
+Wire Wire Line
+	10000 6400 9450 6400
+Wire Wire Line
+	9450 6550 10000 6550
+Wire Wire Line
+	10000 6700 9450 6700
+Wire Wire Line
+	10000 2800 9100 2800
+Wire Wire Line
+	9100 2650 10000 2650
+Wire Wire Line
+	9100 3350 10000 3350
+Wire Wire Line
+	3350 1900 4250 1900
+Wire Wire Line
+	3350 1900 3350 3950
+Wire Wire Line
+	3350 3950 3000 3950
+Wire Wire Line
+	3000 4100 3500 4100
+Wire Wire Line
+	3500 4100 3500 2050
+Wire Wire Line
+	3500 2050 4250 2050
+Wire Wire Line
+	3000 4400 4750 4400
+Wire Wire Line
+	4750 4400 4750 2550
+Wire Wire Line
+	4750 2550 7650 2550
+Wire Wire Line
+	3000 4600 4900 4600
+Wire Wire Line
+	4900 4600 4900 2750
+Wire Wire Line
+	4900 2750 7650 2750
+Wire Wire Line
+	7650 2850 5050 2850
+Wire Wire Line
+	5050 2850 5050 4750
+Wire Wire Line
+	5050 4750 3000 4750
+Wire Wire Line
+	3000 4900 5200 4900
+Wire Wire Line
+	5200 4900 5200 2950
+Wire Wire Line
+	5200 2950 7650 2950
+Wire Wire Line
+	7650 3050 5350 3050
+Wire Wire Line
+	5350 3050 5350 5050
+Wire Wire Line
+	5350 5050 3000 5050
+Wire Wire Line
+	10000 4100 9350 4100
+Wire Wire Line
+	10000 4350 9350 4350
+Wire Wire Line
+	10000 5300 9400 5300
+Wire Wire Line
+	9400 5450 10000 5450
+Wire Wire Line
+	7700 5400 6100 5400
+Wire Wire Line
+	6100 5400 6100 5700
+Wire Wire Line
+	6100 5700 3000 5700
+Wire Wire Line
+	3000 5550 6000 5550
+Wire Wire Line
+	6000 5550 6000 5250
+Wire Wire Line
+	6000 5250 7550 5250
+Wire Wire Line
+	7550 5250 7550 4550
+Wire Wire Line
+	7550 4550 7700 4550
+Wire Wire Line
+	7650 3350 5550 3350
+Wire Wire Line
+	5550 3350 5550 5300
+Wire Wire Line
+	5550 5300 3000 5300
+Wire Wire Line
+	3000 5400 5700 5400
+Wire Wire Line
+	5700 5400 5700 3450
+Wire Wire Line
+	5700 3450 7650 3450
+Wire Wire Line
+	7700 4050 4900 4050
+Connection ~ 4900 4050
+Wire Wire Line
+	7700 4200 5050 4200
+Connection ~ 5050 4200
+Wire Wire Line
+	7700 4400 5350 4400
+Connection ~ 5350 4400
+Wire Wire Line
+	7700 6400 6950 6400
+Wire Wire Line
+	6950 6400 6950 5850
+Wire Wire Line
+	6950 5850 3000 5850
+Wire Wire Line
+	3000 6000 6750 6000
+Wire Wire Line
+	6750 6000 6750 6600
+Wire Wire Line
+	6750 6600 7700 6600
 $EndSCHEMATC
