File: $BenchBudEE.sch (KiCad schematic (older format))
At the start: 0 parts

Commit message: Power
Changed lines of the file:
@@
-EESchema Schematic File Version 2  date 2/8/2014 12:16:58 PM
+EESchema Schematic File Version 2  date 2/8/2014 12:27:29 PM
 LIBS:power
 LIBS:device
@@
 $EndSheet
 $Sheet
-S 7700 3850 1650 1150
+S 7700 4850 1650 1150
 U 52F19DA7
 F0 "Thermocouple" 50
 F1 "Thermocouple.sch" 50
-F2 "TC IN +" I R 9350 4150 60
-F3 "TC IN -" I R 9350 4400 60
-F4 "MOSI" I L 7700 4100 60
-F5 "MISO" O L 7700 4250 60
-F6 "SCLK" I L 7700 4450 60
-F7 "CS_N" I L 7700 4600 60
+F2 "TC IN +" I R 9350 5150 60
+F3 "TC IN -" I R 9350 5400 60
+F4 "MOSI" I L 7700 5100 60
+F5 "MISO" O L 7700 5250 60
+F6 "SCLK" I L 7700 5450 60
+F7 "CS_N" I L 7700 5600 60
 $EndSheet
 $Sheet
-S 7700 5400 1700 1300
+S 7700 6200 1750 700
 U 52F19DBB
 F0 "Relay" 50
 F1 "Relay.sch" 50
-F2 "Din +" I L 7700 5700 60
-F3 "Din -" O L 7700 6000 60
-F4 "NC" B R 9400 5800 60
-F5 "NO" B R 9400 6050 60
-F6 "COM" B R 9400 5550 60
+F2 "Din +" I L 7700 6500 60
+F3 "Din -" O L 7700 6800 60
+F4 "NC" B R 9450 6600 60
+F5 "NO" B R 9450 6850 60
+F6 "COM" B R 9450 6350 60
 $EndSheet
 $Sheet
@@
 $EndSheet
 $Sheet
-S 7700 750  1450 1150
+S 7650 2450 1450 1150
 U 52F19E13
 F0 "Fan" 50
 F1 "Fan.sch" 50
-F2 "Power+" O R 9150 1000 60
-F3 "Power-" I R 9150 1150 60
-F4 "Tach" I R 9150 1300 60
-F5 "TachOUT" O L 7700 1750 60
-F6 "FanIn" I L 7700 900 60
-F7 "Current Measure" O L 7700 1650 60
-F8 "MISO" O L 7700 1150 60
-F9 "MOSI" I L 7700 1050 60
-F10 "SCLK" I L 7700 1250 60
+F2 "Power+" O R 9100 2700 60
+F3 "Power-" I R 9100 2850 60
+F4 "Tach" I R 9100 3000 60
+F5 "TachOUT" O L 7650 3450 60
+F6 "FanIn" I L 7650 2600 60
+F7 "Current Measure" O L 7650 3350 60
+F8 "MISO" O L 7650 2850 60
+F9 "MOSI" I L 7650 2750 60
+F10 "SCLK" I L 7650 2950 60
 $EndSheet
 $Sheet
@@
 $EndSheet
 $Sheet
-S 7700 2150 1700 1300
+S 7700 3850 1700 750
 U 52F19DF1
 F0 "Led_Driver" 50
 F1 "Led_Driver.sch" 50
-F2 "EN" I L 7700 2400 60
-F3 "FREQ" I L 7700 2750 60
-F4 "Strig+" O R 9400 2500 60
-F5 "String-" I R 9400 2750 60
+F2 "EN" I L 7700 4100 60
+F3 "FREQ" I L 7700 4450 60
+F4 "Strig+" O R 9400 4200 60
+F5 "String-" I R 9400 4450 60
 $EndSheet
 $Sheet
-S 4100 1100 1500 1150
+S 4250 1000 1500 1150
 U 52F64696
 F0 "PowerAdjustmentMonitor" 50
 F1 "PowerAdjustmentMonitor.sch" 50
+F2 "V+_ADJ" O R 5750 1150 60
+F3 "V-_ADJ" O R 5750 1300 60
+F4 "3V3_MON" O L 4250 1250 60
+F5 "5V_MON" O L 4250 1100 60
+F6 "V+_ADJ_MON" O L 4250 1900 60
+F7 "V-_ADJ_MON" O L 4250 2050 60
+F8 "V-_CURR_MON" O L 4250 1650 60
+F9 "V+_CURR_MON" O L 4250 1500 60
 $EndSheet
 $EndSCHEMATC
