File: Arduino.sch (KiCad schematic (older format))
At the start: 0 parts

Commit message: Arduino module
Parts:
- added R? (x13): R, ~, symbol R
- added U?: ARDUINO, symbol ARDUINO
Connections:
- net MISO: now also R?.1
- net MOSI: now also R?.1
- net Relay+: now also R?.1
- net Relay-: now also R?.1
- net SCLK: now also R?.1
- net TACH_MEAS: now also R?.1
- new net: R?.2, U?.11 (D0)
- new net: R?.2, U?.12 (D1)
- new net: R?.2, U?.19 (D8)
- new net: R?.2, U?.20 (PWM0)
- new net: R?.2, U?.21 (CS_N)
- new net: R?.2, U?.22 (MOSI)
- new net: R?.2, U?.23 (MISO)
- new net: R?.2, U?.24 (SCK)
- new net: R?.2, U?.5 (A0)
- new net: R?.2, U?.6 (A1)
- new net: R?.2, U?.7 (A2)
- new net: R?.2, U?.8 (A3)
- new net ADC_CS_N: R?.1
- new net CURR_MEAS: R?.1
- new net DAC_CS_N: R?.1
- new net FAN_EN_N: R?.1
- new net GND: R?.2
- new net LED_EN_PWM: R?.1
- new net V+_ADJ_MON: R?.1
- new net V-_ADJ_MON: R?.1
